File: hardware/pcb/areg-reva.kicad_sch (KiCad schematic)
At the start: 100 parts, among them J1 USB4105-GF-A, J2 JST-PH-2 (BATT 3xAA), J3 DM3AT-SF-PEJM5, J4 JST-PH-2 (SPK 8R 50mm), Q1 DMG2301L-7, SW1 B3F-1002 MAIN, SW2 B3F-1002 YES, SW3 B3F-1002 NO, U1 ESP32-S3-WROOM-1-N8R8, U2 MAX98357AETE+T, U3 ICS-43434, U4 TPS63802DLAR, U5 TPD4S014DSQR, U6 USBLC6-2SC6, U7 TPS22918DBVR, U8 IM69D130

Commit message: fix(pcb): wrong ferrite part, plus sourcing-driven passive sizes
The JLCPCB readiness audit (hardware/pcb/jlcpcb-readiness.md, added here)
found a genuine error in the schematic I generated: C1017 is an 0805 part
placed on an 0603 land. It was also the wrong bead in two of the three
positions - FB2/FB3 sit in the class-D speaker path (~0.4 A peak) and had
a 200 mA signal-filter bead on them. Split by role: FB1 -> C1002 (600R,
200 mA), FB2/FB3 -> C14709 (120R, 2 A). Both Basic, both really 0603.

Also: 16 resistor positions move 0402 -> 0603 via a single value-driven
rule (0R/33R/200R/560R/91k/511k). Three of those values have no fee-free
0402 part at all, and the 0402 parts that exist force a minimum-buy worth
more than the loading fee they would dodge. Layout has not started, so
this is free today and a respin later. Inductor gains its LCSC number
(C2849533) after the footprint land was verified against the KiCad file
rather than assumed.

Re-verified after the change: ERC 0 errors (same single justified
warning), netlist still 89 nets, 32 pin-nodes now on 0603.

Order-blocking findings recorded in the readiness doc, NOT silently
fixed - they are the owner's calls: the Bourns detented pot is not in
JLC's catalogue at any tier (hand-solder in Yerevan, the only such part);
TPD4S014 has 96 units in stock with no same-footprint alternative; and
ICS-43434 is ~2 months past its last-time-buy with 5,448 units left,
which is what the IM69D130 alternate footprint already anticipates.

Cost as drawn: ~$214 for 5 assembled boards (~$42.80 each), ~$16.32 each
at 100. Two optional swaps (Q1, D4) would cut $6 of loading fees.

Correction to an earlier assumption, in our favour: JLCPCB does place
through-hole parts now, so the buttons and JST headers are machine-placed
and only the pot is hand-work.

Co-Authored-By: Claude Opus 5 <noreply@anthropic.com>
Claude-Session: https://claude.ai/code/session_019Xbr9SSuqX8c8r7MiLwAbJ
Parts:
- FB1: value BLM18PG601SN1D -> 600R@100MHz 0603 (200mA); LCSC C1017 -> C1002
- FB2, FB3: value BLM18PG601SN1D -> 120R@100MHz 0603 (2A); LCSC C1017 -> C14709
- L1: value 2.2uH VLS6045EX-2R2N -> 2.2uH 6x6mm shielded; LCSC (none) -> C2849533
- R13, R14, R15, R16, R23, R24, R25, R35, R36, R37, R4, R41, R42, R43, R5, R6: footprint Resistor_SMD:R_0402_1005Metric -> Resistor_SMD:R_0603_1608Metric
Changed lines of the file:
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@@
 			(effects (font (size 1.27 1.27)))
 		)
-		(property "Footprint" "Resistor_SMD:R_0402_1005Metric" (at 337.82 144.62 0)
+		(property "Footprint" "Resistor_SMD:R_0603_1608Metric" (at 337.82 144.62 0)
 			(effects (font (size 1.27 1.27)) (hide yes))
 		)
@@
 			(effects (font (size 1.27 1.27)))
 		)
-		(property "Value" "2.2uH VLS6045EX-2R2N" (at 441.96 52.45 0)
+		(property "Value" "2.2uH 6x6mm shielded" (at 441.96 52.45 0)
 			(effects (font (size 1.27 1.27)))
 		)
@@
 			(effects (font (size 1.27 1.27)) (hide yes))
 		)
+		(property "LCSC" "C2849533" (at 441.96 58.45 0)
+			(effects (font (size 1.27 1.27)) (hide yes))
+		)
 		(pin "1")
 		(pin "2")
@@
 			(effects (font (size 1.27 1.27)))
 		)
-		(property "Footprint" "Resistor_SMD:R_0402_1005Metric" (at 480.06 92.55 0)
+		(property "Footprint" "Resistor_SMD:R_0603_1608Metric" (at 480.06 92.55 0)
 			(effects (font (size 1.27 1.27)) (hide yes))
 		)
@@
 			(effects (font (size 1.27 1.27)))
 		)
-		(property "Footprint" "Resistor_SMD:R_0402_1005Metric" (at 480.06 123.03 0)
+		(property "Footprint" "Resistor_SMD:R_0603_1608Metric" (at 480.06 123.03 0)
 			(effects (font (size 1.27 1.27)) (hide yes))
 		)
@@
 			(effects (font (size 1.27 1.27)))
 		)
-		(property "Value" "BLM18PG601SN1D" (at 547.37 67.69 0)
+		(property "Value" "600R@100MHz 0603 (200mA)" (at 547.37 67.69 0)
 			(effects (font (size 1.27 1.27)))
 		)
@@
 			(effects (font (size 1.27 1.27)) (hide yes))
 		)
-		(property "LCSC" "C1017" (at 547.37 73.69 0)
+		(property "LCSC" "C1002" (at 547.37 73.69 0)
 			(effects (font (size 1.27 1.27)) (hide yes))
 		)
@@
 			(effects (font (size 1.27 1.27)))
 		)
-		(property "Footprint" "Resistor_SMD:R_0402_1005Metric" (at 74.93 377.03 0)
+		(property "Footprint" "Resistor_SMD:R_0603_1608Metric" (at 74.93 377.03 0)
 			(effects (font (size 1.27 1.27)) (hide yes))
 		)
@@
 			(effects (font (size 1.27 1.27)))
 		)
-		(property "Footprint" "Resistor_SMD:R_0402_1005Metric" (at 90.17 377.03 0)
+		(property "Footprint" "Resistor_SMD:R_0603_1608Metric" (at 90.17 377.03 0)
 			(effects (font (size 1.27 1.27)) (hide yes))
 		)
@@
 			(effects (font (size 1.27 1.27)))
 		)
-		(property "Footprint" "Resistor_SMD:R_0402_1005Metric" (at 157.48 377.03 0)
+		(property "Footprint" "Resistor_SMD:R_0603_1608Metric" (at 157.48 377.03 0)
 			(effects (font (size 1.27 1.27)) (hide yes))
 		)
@@
 			(effects (font (size 1.27 1.27)))
 		)
-		(property "Footprint" "Resistor_SMD:R_0402_1005Metric" (at 172.72 377.03 0)
+		(property "Footprint" "Resistor_SMD:R_0603_1608Metric" (at 172.72 377.03 0)
 			(effects (font (size 1.27 1.27)) (hide yes))
 		)
@@
 			(effects (font (size 1.27 1.27)))
 		)
-		(property "Footprint" "Resistor_SMD:R_0402_1005Metric" (at 353.06 377.03 0)
+		(property "Footprint" "Resistor_SMD:R_0603_1608Metric" (at 353.06 377.03 0)
 			(effects (font (size 1.27 1.27)) (hide yes))
 		)
@@
 			(effects (font (size 1.27 1.27)))
 		)
-		(property "Footprint" "Resistor_SMD:R_0402_1005Metric" (at 367.03 377.03 0)
+		(property "Footprint" "Resistor_SMD:R_0603_1608Metric" (at 367.03 377.03 0)
 			(effects (font (size 1.27 1.27)) (hide yes))
 		)
@@
 			(effects (font (size 1.27 1.27)))
 		)
-		(property "Footprint" "Resistor_SMD:R_0402_1005Metric" (at 382.27 377.03 0)
+		(property "Footprint" "Resistor_SMD:R_0603_1608Metric" (at 382.27 377.03 0)
 			(effects (font (size 1.27 1.27)) (hide yes))
 		)
@@
 			(effects (font (size 1.27 1.27)))
 		)
-		(property "Footprint" "Resistor_SMD:R_0402_1005Metric" (at 637.54 317.34 0)
+		(property "Footprint" "Resistor_SMD:R_0603_1608Metric" (at 637.54 317.34 0)
 			(effects (font (size 1.27 1.27)) (hide yes))
 		)
@@
 			(effects (font (size 1.27 1.27)))
 		)
-		(property "Footprint" "Resistor_SMD:R_0402_1005Metric" (at 652.78 317.34 0)
+		(property "Footprint" "Resistor_SMD:R_0603_1608Metric" (at 652.78 317.34 0)
 			(effects (font (size 1.27 1.27)) (hide yes))
 		)
@@
 			(effects (font (size 1.27 1.27)))
 		)
-		(property "Footprint" "Resistor_SMD:R_0402_1005Metric" (at 668.02 317.34 0)
+		(property "Footprint" "Resistor_SMD:R_0603_1608Metric" (at 668.02 317.34 0)
 			(effects (font (size 1.27 1.27)) (hide yes))
 		)
@@
 			(effects (font (size 1.27 1.27)))
 		)
-		(property "Value" "BLM18PG601SN1D" (at 742.95 338.2 0)
+		(property "Value" "120R@100MHz 0603 (2A)" (at 742.95 338.2 0)
 			(effects (font (size 1.27 1.27)))
 		)
@@
 			(effects (font (size 1.27 1.27)) (hide yes))
 		)
-		(property "LCSC" "C1017" (at 742.95 344.2 0)
+		(property "LCSC" "C14709" (at 742.95 344.2 0)
 			(effects (font (size 1.27 1.27)) (hide yes))
 		)
@@
 			(effects (font (size 1.27 1.27)))
 		)
-		(property "Value" "BLM18PG601SN1D" (at 756.92 338.2 0)
+		(property "Value" "120R@100MHz 0603 (2A)" (at 756.92 338.2 0)
 			(effects (font (size 1.27 1.27)))
 		)
@@
 			(effects (font (size 1.27 1.27)) (hide yes))
 		)
-		(property "LCSC" "C1017" (at 756.92 344.2 0)
+		(property "LCSC" "C14709" (at 756.92 344.2 0)
 			(effects (font (size 1.27 1.27)) (hide yes))
 		)
@@
 			(effects (font (size 1.27 1.27)))
 		)
-		(property "Footprint" "Resistor_SMD:R_0402_1005Metric" (at 157.48 467.2 0)
+		(property "Footprint" "Resistor_SMD:R_0603_1608Metric" (at 157.48 467.2 0)
 			(effects (font (size 1.27 1.27)) (hide yes))
 		)
@@
 			(effects (font (size 1.27 1.27)))
 		)
-		(property "Footprint" "Resistor_SMD:R_0402_1005Metric" (at 195.58 467.2 0)
+		(property "Footprint" "Resistor_SMD:R_0603_1608Metric" (at 195.58 467.2 0)
 			(effects (font (size 1.27 1.27)) (hide yes))
 		)
@@
 			(effects (font (size 1.27 1.27)))
 		)
-		(property "Footprint" "Resistor_SMD:R_0402_1005Metric" (at 232.41 467.2 0)
-			(effects (font (size 1.27 1.27)) (hide yes))
-		)
+		(property "Footprint" "Resistor_SMD:R_0603_1608Metric" (at 232.41 467.2 0)
+			(effects (font (size 1.27 1.27)) (hide yes))
+		)

Commit message: feat(pcb): rev-A board placed, 4-layer, 0 DRC errors - 11 pads still open
Independently re-verified before commit: kicad-cli pcb drc --severity-all
--schematic-parity => 0 errors, 16 warnings (silkscreen over pads at 0402
density, justified), schematic parity 0, 11 unconnected pads. Board is
74 x 62 mm, 100/100 footprints top-side, 824 tracks, 340 vias.

NOT a finished board, and not claimed as one. 71 of 74 signal nets route
fully; the 11 open pads are listed by ref/pin/net in phase2-status.md and
sit inside the 0.5 mm-pitch amp, the 0.4 mm-pitch USB protection IC, the
interleaved USB-C D+/D- pads and the mic pocket - push-and-shove work an
interactive router does in minutes and a headless one cannot.

Three real defects were caught in the process, none of which ERC could
have found:

1. The TPS63802's exposed thermal pad was MISSING FROM THE SYMBOL
   ENTIRELY. It is the main GND return and the only heat path for a 2 A
   buck-boost, so the fabricated board would have had it floating. Found
   because the layout had a copper pad with no net to route - ERC cannot
   flag a pin that was never declared. Every exposed pad on the board was
   then audited by script: U1, U2, U4, U5 all carry GND with a via in
   pad; U6/U7 (SOT-23-6) and the LGA mics have none by construction.

2. Schematic parity was reported as 0 by earlier passes because that
   section of the report is empty unless --schematic-parity is actually
   passed. Run properly it was 157: 112 unqualified footprint IDs and 45
   MISSING LCSC FIELDS - a JLCPCB BOM with 45 blank part numbers. Fixed,
   and the 12 test pads are now excluded from the BOM at source.

3. The first inner-plane plan carved VSYS/VBUS islands that SPLIT THE
   +3V3 PLANE IN TWO - a severed main rail. Visible only in the layer
   plots, not in the 3D render. In2.Cu is now one solid plane.

Board grew from the 60x50 target to 74x62 because the unshrinkable parts
are ~1,200 mm2 of courtyard on a single assembly side; +$0.11/board.

Befor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
Parts:
- TP1, TP10, TP11, TP12, TP2, TP3, TP4, TP5, TP6, TP7, TP8, TP9: now left out of the parts list
Connections:
- net GND: now also U4.11 (PAD)
